Commit message: Update URDF

File: urdf/spotmicroai.urdf (robot description, URDF)
Before this commit: robot SpotMicroAI, 24 links, 23 joints
Links:
- added link imu_link, mass 0.001
- added link lidar_link, mass 0.50; collision box size=0.0985 0.0577 0.07; visual mesh filename=package://spotmicro_description/meshes/stl/rplidar_main.STL scale=0.001 0.001 0.001
Joints:
- added joint base_lidar: type fixed, parent base_link, child lidar_link, origin xyz=0 0 0.035
- added joint imu_joint: type fixed, parent base_link, child imu_link

File: urdf/spotmicroai.urdf.xacro (robot description, xacro)
@@ -1,4 +1,7 @@
 <?xml version="1.0" encoding="UTF-8"?>
 <robot xmlns:xacro="http://www.ros.org/wiki/xacro" name="SpotMicroAI">
+   <xacro:include filename="$(find spotmicro_description)/urdf/include/accessories.urdf.xacro"/>
+   <xacro:include filename="$(find spotmicro_description)/urdf/include/spotmicroai_leg.urdf.xacro"/>
+   <xacro:include filename="$(optenv SPOT_URDF_EXTRAS empty.urdf)" />
    <material name="yellow">
       <color rgba="0.92 0.83 0.0 1" />
@@ -10,205 +13,4 @@
       <color rgba="0.6 0.6 0.6 1" />
    </material>
-   <!-- Params -->
-   <xacro:property name="body_length" value="0.140" />
-   <xacro:property name="body_width" value="0.110" />
-   <xacro:property name="body_height" value="0.070" />
-   <xacro:property name="lidar_length" value="0.0985" />
-   <xacro:property name="lidar_width" value="0.0577" />
-   <xacro:property name="lidar_height" value="0.070" />
-   <xacro:property name="front_length" value="0.058" />
-   <xacro:property name="rear_length" value="0.040" />
-   <xacro:property name="shoulder_length" value="0.044" />
-   <xacro:property name="shoulder_width" value="0.038" />
-   <xacro:property name="leg_length" value="0.109" />
-   <xacro:property name="foot_length" value="0.13" />
-   <xacro:property name="toe_radius" value="0.020" />
-   <!--  <xacro:property name="toe_radius" value="0.014" /> -->
-   <xacro:property name="toe_width" value="0.020" />
-   <xacro:property name="shift" value="0.055" />
-   <xacro:property name="shiftx" value="0.093" />
-   <xacro:property name="shifty" value="0.0395" />
-   <!-- Macros -->
-   <xacro:macro name="gen_shoulder" params="name left">
-      <link name="${name}">
-         <visual>
-            <xacro:if value="${left}">
-               <geometry>
-                  <mesh filename="package://spotmicro_description/meshes/stl/lshoulder.stl" scale="0.001 0.001 0.001" />
-               </geometry>
-               <origin rpy="0 0 3.1416" xyz="0.135 0.0163 -0.0195" />
-            </xacro:if>
-            <xacro:unless value="${left}">
-               <geometry>
-                  <mesh filename="package://spotmicro_description/meshes/stl/rshoulder.stl" scale="0.001 0.001 0.001" />
-               </geometry>
-               <origin rpy="0 0 3.1416" xyz="0.135 0.0938 -0.0205" />
-            </xacro:unless>
-            <material name="black" />
-         </visual>
-         <collision>
-            <geometry>
-               <box size="${shoulder_length} ${shoulder_width} ${body_height}" />
-            </geometry>
-            <origin rpy="0 0 0" xyz="0 0 0" />
-         </collision>
-         <inertial>
-            <mass value="0.10" />
-            <inertia ixx="100" ixy="0" ixz="0" iyy="100" iyz="0" izz="100" />
-         </inertial>
-      </link>
-   </xacro:macro>
-   <xacro:macro name="gen_shoulder_joint" params="pos shiftx shifty">
-      <joint name="${pos}_shoulder" type="revolute">
-         <parent link="base_link" />
-         <child link="${pos}_shoulder_link" />
-         <axis xyz="1 0 0" />
-         <origin rpy="0 0 0" xyz="${shiftx} ${shifty} 0" />
-         <limit effort="1000.0" lower="-0.548" upper="0.548" velocity="0.7" />
-         <dynamics damping="0.0" friction="0.5" />
-      </joint>
-   </xacro:macro>
-   <xacro:macro name="gen_leg" params="name left">
-      <link name="${name}_cover">
-         <visual>
-            <xacro:if value="${left}">
-               <geometry>
-                  <mesh filename="package://spotmicro_description/meshes/stl/larm_cover.stl" scale="0.001 0.001 0.001" />
-               </geometry>
-               <origin rpy="0 0 3.1416" xyz="0.134 -0.04 -0.0095" />
-            </xacro:if>
-            <xacro:unless value="${left}">
-               <geometry>
-                  <mesh filename="package://spotmicro_description/meshes/stl/rarm_cover.stl" scale="0.001 0.001 0.001" />
-               </geometry>
-               <origin rpy="0 0 3.1416" xyz="0.134 0.149 -0.0095" />
-            </xacro:unless>
-            <material name="yellow" />
-         </visual>
-      </link>
-      <link name="${name}">
-         <visual>
-            <xacro:if value="${left}">
-               <geometry>
-                  <mesh filename="package://spotmicro_description/meshes/stl/larm.stl" scale="0.001 0.001 0.001" />
-               </geometry>
-               <origin rpy="0 0 3.1416" xyz="0.134 -0.04 -0.0095" />
-            </xacro:if>
-            <xacro:unless value="${left}">
-               <geometry>
-                  <mesh filename="package://spotmicro_description/meshes/stl/rarm.stl" scale="0.001 0.001 0.001" />
-               </geometry>
-               <origin rpy="0 0 3.1416" xyz="0.134 0.149 -0.0095" />
-            </xacro:unless>
-            <material name="black" />
-         </visual>
-         <collision>
-            <origin rpy="0.0 0.0 0.0" xyz="0.0 0.0 -0.050" />
-            <geometry>
-               <box size="0.028 0.036 ${leg_length}" />
-            </geometry>
-         </collision>
-         <inertial>
-            <mass value="0.15" />
-            <inertia ixx="1000" ixy="0" ixz="0" iyy="1000" iyz="0" izz="1000" />
-         </inertial>
-      </link>
-      <gazebo reference="${name}_cover">
-         <material>Gazebo/ZincYellow</material>
-      </gazebo>
-   </xacro:macro>
-   <xacro:macro name="gen_leg_joint" params="pos shift">
-      <joint name="${pos}_leg" type="revolute">
-         <parent link="${pos}_shoulder_link" />
-         <child link="${pos}_leg_link" />
-         <axis xyz="0 1 0" />
-         <origin rpy="0 0 0" xyz="0 ${shift} 0" />
-         <limit effort="1000.0" lower="-2.666" upper="1.548" velocity="0.5" />
-         <dynamics damping="0.0" friction="0.0" />
-      </joint>
-      <joint name="${pos}_leg_cover_joint" type="fixed">
-         <parent link="${pos}_leg_link" />
-         <child link="${pos}_leg_link_cover" />
-         <origin xyz="0 0 0" />
-      </joint>
-   </xacro:macro>
-   <xacro:macro name="gen_foot" params="name left">
-      <link name="${name}">
-         <visual>
-            <xacro:if value="${left}">
-               <geometry>
-                  <mesh filename="package://spotmicro_description/meshes/stl/lfoot.stl" scale="0.001 0.001 0.001" />
-               </geometry>
-               <origin rpy="0 0 3.1416 " xyz="0.1195 -0.04 0.099" />
-            </xacro:if>
-            <xacro:unless value="${left}">
-               <geometry>
-                  <mesh filename="package://spotmicro_description/meshes/stl/rfoot.stl" scale="0.001 0.001 0.001" />
-               </geometry>
-               <origin rpy="0 0 3.1416" xyz="0.1195 0.149 0.099" />
-            </xacro:unless>
-            <material name="black" />
-         </visual>
-         <collision>
-            <geometry>
-               <box size="0.026 0.020 ${foot_length}" />
-            </geometry>
-            <origin rpy="0.0 0.0 0.0" xyz="0.0 0.0 -0.050" />
-         </collision>
-         <inertial>
-            <mass value="0.1" />
-            <inertia ixx="1000" ixy="0" ixz="0" iyy="1000" iyz="0" izz="1000" />
-         </inertial>
-      </link>
-   </xacro:macro>
-   <xacro:macro name="gen_foot_joint" params="pos">
-      <joint name="${pos}_foot" type="revolute">
-         <parent link="${pos}_leg_link" />
-         <child link="${pos}_foot_link" />
-         <axis xyz="0 1 0" />
-         <origin rpy="0 0 0" xyz="0.014 0 -${leg_length}" />
-         <limit effort="1000.0" lower="-0.1" upper="2.59" velocity="0.5" />
-         <dynamics damping="0.0" friction="0.5" />
-      </joint>
-   </xacro:macro>
-   <xacro:macro name="gen_toe" params="name">
-      <link name="${name}">
-         <visual>
-            <geometry>
-               <mesh filename="package://spotmicro_description/meshes/stl/foot.stl" scale="0.001 0.001 0.001" />
-            </geometry>
-            <origin rpy="0 0.40010 0" xyz="0 -0.01 0.015" />
-            <material name="grey" />
-         </visual>
-         <collision>
-            <geometry>
-               <sphere radius="${toe_radius}" />
-            </geometry>
-            <origin rpy="0 0 0" xyz="0 0 0" />
-            <contact_coefficients mu="1.1" />
-         </collision>
-         <inertial>
-            <mass value="0.05" />
-            <inertia ixx="1000" ixy="0" ixz="0" iyy="1000" iyz="0" izz="1000" />
-         </inertial>
-      </link>
-   </xacro:macro>
-   <xacro:macro name="gen_toe_joint" params="pos">
-      <joint name="${pos}_toe" type="fixed">
-         <parent link="${pos}_foot_link" />
-         <child link="${pos}_toe_link" />
-         <origin xyz="0 0 -${foot_length}" />
-      </joint>
-   </xacro:macro>
-   <xacro:macro name="gen_full_leg_joint" params="pos shiftx shifty shift left">
-      <xacro:gen_shoulder name="${pos}_shoulder_link" left="${left}" />
-      <xacro:gen_leg name="${pos}_leg_link" left="${left}" />
-      <xacro:gen_foot name="${pos}_foot_link" left="${left}" />
-      <xacro:gen_toe name="${pos}_toe_link" />
-      <xacro:gen_shoulder_joint pos="${pos}" shiftx="${shiftx}" shifty="${shifty}" />
-      <xacro:gen_leg_joint pos="${pos}" shift="${shift}" />
-      <xacro:gen_foot_joint pos="${pos}" />
-      <xacro:gen_toe_joint pos="${pos}" />
-   </xacro:macro>
    <!-- Robot Body -->
    <link name="base_link"/>
@@ -293,3 +95,21 @@
    <xacro:gen_full_leg_joint pos="rear_left" shiftx="-${shiftx}" shifty="${shifty}" shift="${shift}" left="true" />
    <xacro:gen_full_leg_joint pos="rear_right" shiftx="-${shiftx}" shifty="-${shifty}" shift="-${shift}" left="false" />
+   <!-- Optional custom includes. -->
+   <gazebo>
+      <plugin name="p3d_base_controller" filename="libgazebo_ros_p3d.so">
+         <alwaysOn>true</alwaysOn>
+         <updateRate>10.0</updateRate>
+         <bodyName>base_link</bodyName>
+         <topicName>odom/ground_truth</topicName>
+         <gaussianNoise>0.01</gaussianNoise>
+         <frameName>world</frameName>
+         <xyzOffsets>0 0 0</xyzOffsets>
+         <rpyOffsets>0 0 0</rpyOffsets>
+      </plugin>
+   </gazebo>
+   <gazebo>
+      <plugin name="gazebo_ros_control" filename="libgazebo_ros_control.so">
+         <legacyModeNS>true</legacyModeNS>
+      </plugin>
+   </gazebo>
 </robot>
