Commit message: Make the legs stabilize correctly

File: urdf/spotmicroai.urdf (robot description, URDF)
Before this commit: robot SpotMicroAI, 24 links, 23 joints
Links:
- added link imu_link, mass 0.001
- link base_inertia: mass 2.80 -> 2.8
- link front_left_foot_link: geometry collision box size=0.026 0.02 0.125; visual mesh filename=package://spotmicro_description/meshes/stl/lfoot.stl scale=0.001 0.001 0.001
- link front_left_shoulder_link: mass 0.10 -> 0.1
- link front_left_toe_link: geometry collision sphere radius=0.015; visual mesh filename=package://spotmicro_description/meshes/stl/foot.stl scale=0.001 0.001 0.001
- link front_link: mass 0.20 -> 0.2
- link front_right_foot_link: geometry collision box size=0.026 0.02 0.125; visual mesh filename=package://spotmicro_description/meshes/stl/rfoot.stl scale=0.001 0.001 0.001
- link front_right_shoulder_link: mass 0.10 -> 0.1
- link front_right_toe_link: geometry collision sphere radius=0.015; visual mesh filename=package://spotmicro_description/meshes/stl/foot.stl scale=0.001 0.001 0.001
- link rear_left_foot_link: geometry collision box size=0.026 0.02 0.125; visual mesh filename=package://spotmicro_description/meshes/stl/lfoot.stl scale=0.001 0.001 0.001
- link rear_left_shoulder_link: mass 0.10 -> 0.1
- link rear_left_toe_link: geometry collision sphere radius=0.015; visual mesh filename=package://spotmicro_description/meshes/stl/foot.stl scale=0.001 0.001 0.001
- link rear_link: mass 0.20 -> 0.2
- link rear_right_foot_link: geometry collision box size=0.026 0.02 0.125; visual mesh filename=package://spotmicro_description/meshes/stl/rfoot.stl scale=0.001 0.001 0.001
- link rear_right_shoulder_link: mass 0.10 -> 0.1
- link rear_right_toe_link: geometry collision sphere radius=0.015; visual mesh filename=package://spotmicro_description/meshes/stl/foot.stl scale=0.001 0.001 0.001
Joints:
- added joint imu_joint: type fixed, parent base_link, child imu_link
- joint front_left_foot: limit lower=-0.1 upper=2.59 effort=1000.0 velocity=0.5 -> lower=-1.7929 upper=0.254801 effort=100.0 velocity=0.5
- joint front_left_leg: limit lower=-2.666 upper=1.548 effort=1000.0 velocity=0.5 -> lower=-2.666 upper=1.548 effort=100.0 velocity=0.5
- joint front_left_shoulder: limit lower=-0.548 upper=0.548 effort=1000.0 velocity=0.7 -> lower=-0.548 upper=0.548 effort=100.0 velocity=0.7
- joint front_left_toe: origin xyz=0 0 -0.13 -> xyz=0 0 -0.125
- joint front_right_foot: limit lower=-0.1 upper=2.59 effort=1000.0 velocity=0.5 -> lower=-1.7929 upper=0.254801 effort=100.0 velocity=0.5
- joint front_right_leg: limit lower=-2.666 upper=1.548 effort=1000.0 velocity=0.5 -> lower=-2.666 upper=1.548 effort=100.0 velocity=0.5
- joint front_right_shoulder: limit lower=-0.548 upper=0.548 effort=1000.0 velocity=0.7 -> lower=-0.548 upper=0.548 effort=100.0 velocity=0.7
- joint front_right_toe: origin xyz=0 0 -0.13 -> xyz=0 0 -0.125
- joint rear_left_foot: limit lower=-0.1 upper=2.59 effort=1000.0 velocity=0.5 -> lower=-1.7929 upper=0.254801 effort=100.0 velocity=0.5
- joint rear_left_leg: limit lower=-2.666 upper=1.548 effort=1000.0 velocity=0.5 -> lower=-2.666 upper=1.548 effort=100.0 velocity=0.5
- joint rear_left_shoulder: limit lower=-0.548 upper=0.548 effort=1000.0 velocity=0.7 -> lower=-0.548 upper=0.548 effort=100.0 velocity=0.7
- joint rear_left_toe: origin xyz=0 0 -0.13 -> xyz=0 0 -0.125
- joint rear_right_foot: limit lower=-0.1 upper=2.59 effort=1000.0 velocity=0.5 -> lower=-1.7929 upper=0.254801 effort=100.0 velocity=0.5
- joint rear_right_leg: limit lower=-2.666 upper=1.548 effort=1000.0 velocity=0.5 -> lower=-2.666 upper=1.548 effort=100.0 velocity=0.5
- joint rear_right_shoulder: limit lower=-0.548 upper=0.548 effort=1000.0 velocity=0.7 -> lower=-0.548 upper=0.548 effort=100.0 velocity=0.7
- joint rear_right_toe: origin xyz=0 0 -0.13 -> xyz=0 0 -0.125

File: urdf/spotmicroai.urdf.xacro (robot description, xacro)
@@ -1,4 +1,6 @@
 <?xml version="1.0" encoding="UTF-8"?>
 <robot xmlns:xacro="http://www.ros.org/wiki/xacro" name="SpotMicroAI">
+   <xacro:include filename="include/constants.urdf.xacro"/>
+   <xacro:include filename="include/inertias.urdf.xacro"/>
    <material name="yellow">
       <color rgba="0.92 0.83 0.0 1" />
@@ -10,23 +12,4 @@
       <color rgba="0.6 0.6 0.6 1" />
    </material>
-   <!-- Params -->
-   <xacro:property name="body_length" value="0.140" />
-   <xacro:property name="body_width" value="0.110" />
-   <xacro:property name="body_height" value="0.070" />
-   <xacro:property name="lidar_length" value="0.0985" />
-   <xacro:property name="lidar_width" value="0.0577" />
-   <xacro:property name="lidar_height" value="0.070" />
-   <xacro:property name="front_length" value="0.058" />
-   <xacro:property name="rear_length" value="0.040" />
-   <xacro:property name="shoulder_length" value="0.044" />
-   <xacro:property name="shoulder_width" value="0.038" />
-   <xacro:property name="leg_length" value="0.109" />
-   <xacro:property name="foot_length" value="0.13" />
-   <xacro:property name="toe_radius" value="0.020" />
-   <!--  <xacro:property name="toe_radius" value="0.014" /> -->
-   <xacro:property name="toe_width" value="0.020" />
-   <xacro:property name="shift" value="0.055" />
-   <xacro:property name="shiftx" value="0.093" />
-   <xacro:property name="shifty" value="0.0395" />
    <!-- Macros -->
    <xacro:macro name="gen_shoulder" params="name left">
@@ -53,8 +36,5 @@
             <origin rpy="0 0 0" xyz="0 0 0" />
          </collision>
-         <inertial>
-            <mass value="0.10" />
-            <inertia ixx="100" ixy="0" ixz="0" iyy="100" iyz="0" izz="100" />
-         </inertial>
+         <xacro:inertial_cuboid mass="0.10" x_length="${shoulder_length}" y_length="${shoulder_width}" z_length="${body_height}"/>
       </link>
    </xacro:macro>
@@ -65,7 +45,16 @@
          <axis xyz="1 0 0" />
          <origin rpy="0 0 0" xyz="${shiftx} ${shifty} 0" />
-         <limit effort="1000.0" lower="-0.548" upper="0.548" velocity="0.7" />
-         <dynamics damping="0.0" friction="0.5" />
-      </joint>
+         <limit effort="100.0" lower="-0.548" upper="0.548" velocity="0.7" />
+      </joint>
+      <transmission name="${pos}_shoulder_trans">
+         <type>transmission_interface/SimpleTransmission</type>
+         <joint name="${pos}_shoulder">
+               <hardwareInterface>hardware_interface/EffortJointInterface</hardwareInterface>
+         </joint>
+         <actuator name="${pos}_shoulder_actuator">
+               <hardwareInterface>hardware_interface/EffortJointInterface</hardwareInterface>
+               <mechanicalReduction>1</mechanicalReduction>
+         </actuator>
+      </transmission>
    </xacro:macro>
    <xacro:macro name="gen_leg" params="name left">
@@ -104,13 +93,12 @@
          </visual>
          <collision>
-            <origin rpy="0.0 0.0 0.0" xyz="0.0 0.0 -0.050" />
-            <geometry>
-               <box size="0.028 0.036 ${leg_length}" />
+            <origin rpy="0 0 0" xyz="0 0 -0.050" />
+            <geometry>
+               <box size="${leg_height} ${leg_width} ${leg_length}" />
             </geometry>
          </collision>
-         <inertial>
-            <mass value="0.15" />
-            <inertia ixx="1000" ixy="0" ixz="0" iyy="1000" iyz="0" izz="1000" />
-         </inertial>
+         <xacro:inertial_cuboid_with_pose mass="${leg_mass}" x_length="${leg_height}" y_length="${leg_width}" z_length="${leg_length}">
+            <origin rpy="0 0 0" xyz="0 0 -0.050" />
+         </xacro:inertial_cuboid_with_pose>
       </link>
       <gazebo reference="${name}_cover">
@@ -124,7 +112,16 @@
          <axis xyz="0 1 0" />
          <origin rpy="0 0 0" xyz="0 ${shift} 0" />
-         <limit effort="1000.0" lower="-2.666" upper="1.548" velocity="0.5" />
-         <dynamics damping="0.0" friction="0.0" />
-      </joint>
+         <limit effort="100.0" lower="-2.666" upper="1.548" velocity="0.5" />
+      </joint>
+      <transmission name="${pos}_leg_trans">
+         <type>transmission_interface/SimpleTransmission</type>
+         <joint name="${pos}_leg">
+               <hardwareInterface>hardware_interface/EffortJointInterface</hardwareInterface>
+         </joint>
+         <actuator name="${pos}_leg_actuator">
+               <hardwareInterface>hardware_interface/EffortJointInterface</hardwareInterface>
+               <mechanicalReduction>1</mechanicalReduction>
+         </actuator>
+      </transmission>
       <joint name="${pos}_leg_cover_joint" type="fixed">
          <parent link="${pos}_leg_link" />
@@ -152,13 +149,20 @@
          <collision>
             <geometry>
-               <box size="0.026 0.020 ${foot_length}" />
-            </geometry>
-            <origin rpy="0.0 0.0 0.0" xyz="0.0 0.0 -0.050" />
+               <box size="${foot_height} ${foot_width} ${foot_length}" />
+            </geometry>
+            <origin rpy="0 0 0" xyz="0 0 -0.050" />
          </collision>
-         <inertial>
-            <mass value="0.1" />
-            <inertia ixx="1000" ixy="0" ixz="0" iyy="1000" iyz="0" izz="1000" />
-         </inertial>
-      </link>
+         <xacro:inertial_cuboid_with_pose mass="${foot_mass}" x_length="${foot_height}" y_length="${foot_width}" z_length="${foot_length}">
+            <origin rpy="0 0 0" xyz="0 0 -0.050" />
+         </xacro:inertial_cuboid_with_pose>
+      </link>
+      <gazebo reference="${name}">
+         <kp>100000.0</kp>
+         <kd>1.0</kd>
+         <mu1>0.8</mu1>
+         <mu2>0.8</mu2>
+         <maxVel>0.0</maxVel>
+         <minDepth>0.001</minDepth>
+      </gazebo>
    </xacro:macro>
    <xacro:macro name="gen_foot_joint" params="pos">
@@ -168,7 +172,16 @@
          <axis xyz="0 1 0" />
          <origin rpy="0 0 0" xyz="0.014 0 -${leg_length}" />
-         <limit effort="1000.0" lower="-0.1" upper="2.59" velocity="0.5" />
-         <dynamics damping="0.0" friction="0.5" />
-      </joint>
+         <limit effort="100.0" lower="-1.7929" upper="0.254801" velocity="0.5" />
+      </joint>
+      <transmission name="${pos}_foot_trans">
+         <type>transmission_interface/SimpleTransmission</type>
+         <joint name="${pos}_foot">
+               <hardwareInterface>hardware_interface/EffortJointInterface</hardwareInterface>
+         </joint>
+         <actuator name="${pos}_foot_actuator">
+               <hardwareInterface>hardware_interface/EffortJointInterface</hardwareInterface>
+               <mechanicalReduction>1</mechanicalReduction>
+         </actuator>
+      </transmission>
    </xacro:macro>
    <xacro:macro name="gen_toe" params="name">
@@ -178,5 +191,5 @@
                <mesh filename="package://spotmicro_description/meshes/stl/foot.stl" scale="0.001 0.001 0.001" />
             </geometry>
-            <origin rpy="0 0.40010 0" xyz="0 -0.01 0.015" />
+            <origin rpy="0 0.40010 0" xyz="0 -0.01 0.005" />
             <material name="grey" />
          </visual>
@@ -188,9 +201,14 @@
             <contact_coefficients mu="1.1" />
          </collision>
-         <inertial>
-            <mass value="0.05" />
-            <inertia ixx="1000" ixy="0" ixz="0" iyy="1000" iyz="0" izz="1000" />
-         </inertial>
-      </link>
+         <xacro:inertial_sphere mass="${toe_mass}" diameter="${toe_radius}"/>
+      </link>
+      <gazebo reference="${name}">
+         <kp>100000.0</kp>
+         <kd>1.0</kd>
+         <mu1>1.0</mu1>
+         <mu2>1.0</mu2>
+         <maxVel>0.0</maxVel>
+         <minDepth>0.001</minDepth>
+      </gazebo>
    </xacro:macro>
    <xacro:macro name="gen_toe_joint" params="pos">
@@ -227,8 +245,7 @@
          <origin rpy="0 0 3.1416" xyz="0 0 0" />
       </collision>
-      <inertial>
-         <mass value="2.80" />
-         <inertia ixx="100" ixy="0" ixz="0" iyy="100" iyz="0" izz="100" />
-      </inertial>
+      <xacro:inertial_cuboid_with_pose mass="${body_mass}" x_length="${body_length}" y_length="${body_width}" z_length="${body_height}">
+         <origin rpy="0 0 3.1416" xyz="0 0 0" />
+      </xacro:inertial_cuboid_with_pose>
    </link>
    <joint name="base_inertia_joint" type="fixed">
@@ -250,8 +267,7 @@
          <origin rpy="0 0 0" xyz="-0.135 0 0" />
       </collision>
-      <inertial>
-         <mass value="0.20" />
-         <inertia ixx="100" ixy="0" ixz="0" iyy="100" iyz="0" izz="100" />
-      </inertial>
+      <xacro:inertial_cuboid_with_pose mass="0.20" x_length="${rear_length}" y_length="${body_width}" z_length="${body_height}">
+         <origin rpy="0 0 0" xyz="-0.135 0 0" />
+      </xacro:inertial_cuboid_with_pose>
    </link>
    <joint name="base_rear" type="fixed">
@@ -276,8 +292,7 @@
          <origin rpy="0 0 0" xyz="0.135 0 0" />
       </collision>
-      <inertial>
-         <mass value="0.20" />
-         <inertia ixx="100" ixy="0" ixz="0" iyy="100" iyz="0" izz="100" />
-      </inertial>
+      <xacro:inertial_cuboid_with_pose mass="0.20" x_length="${front_length}" y_length="${body_width}" z_length="${body_height}">
+         <origin rpy="0 0 0" xyz="0.135 0 0" />
+      </xacro:inertial_cuboid_with_pose>
    </link>
    <gazebo reference="front_link">
@@ -289,7 +304,28 @@
    </joint>
    <!-- create Legs -->
-   <xacro:gen_full_leg_joint pos="front_left" shiftx="${shiftx}" shifty="${shifty}" shift="${shift}" left="true" />
-   <xacro:gen_full_leg_joint pos="front_right" shiftx="${shiftx}" shifty="-${shifty}" shift="-${shift}" left="false" />
-   <xacro:gen_full_leg_joint pos="rear_left" shiftx="-${shiftx}" shifty="${shifty}" shift="${shift}" left="true" />
-   <xacro:gen_full_leg_joint pos="rear_right" shiftx="-${shiftx}" shifty="-${shifty}" shift="-${shift}" left="false" />
+   <xacro:gen_full_leg_joint pos="front_left"  shiftx=" ${shiftx}" shifty=" ${shifty}" shift=" ${shift}" left="true"  />
+   <xacro:gen_full_leg_joint pos="front_right" shiftx=" ${shiftx}" shifty="-${shifty}" shift="-${shift}" left="false" />
+   <xacro:gen_full_leg_joint pos="rear_left"   shiftx="-${shiftx}" shifty=" ${shifty}" shift=" ${shift}" left="true"  />
+   <xacro:gen_full_leg_joint pos="rear_right"  shiftx="-${shiftx}" shifty="-${shifty}" shift="-${shift}" left="false" />
+   <!-- Optional custom includes. -->
+   <xacro:include filename="$(optenv SPOT_URDF_EXTRAS empty.urdf)" />
+   <xacro:include filename="include/accessories.urdf.xacro" />
+   <!-- Gazebo plugins -->
+   <gazebo>
+      <plugin name="p3d_base_controller" filename="libgazebo_ros_p3d.so">
+            <alwaysOn>true</alwaysOn>
+            <updateRate>10.0</updateRate>
+            <bodyName>base_link</bodyName>
+            <topicName>odom/ground_truth</topicName>
+            <gaussianNoise>0.01</gaussianNoise>
+            <frameName>world</frameName>
+            <xyzOffsets>0 0 0</xyzOffsets>
+            <rpyOffsets>0 0 0</rpyOffsets>
+        </plugin>
+    </gazebo>
+    <gazebo>
+        <plugin name="gazebo_ros_control" filename="libgazebo_ros_control.so">
+            <legacyModeNS>true</legacyModeNS>
+        </plugin>
+    </gazebo>
 </robot>

Commit message: Update URDF - Add Realsense and IMU

File: urdf/spotmicroai.urdf (robot description, URDF)
Before this commit: robot SpotMicroAI, 24 links, 23 joints
Links:
- added link d435_bottom_screw_frame
- added link d435_color_frame
- added link d435_color_optical_frame
- added link d435_depth_frame
- added link d435_depth_optical_frame
- added link d435_infra1_frame
- added link d435_infra1_optical_frame
- added link d435_infra2_frame
- added link d435_infra2_optical_frame
- added link d435_link, mass 0.072; collision box size=0.02505 0.09 0.025; visual mesh filename=package://realsense2_description/meshes/d435.dae
- added link imu_link
- link front_link: geometry collision box size=0.058 0.11 0.07; visual mesh filename=package://spotmicro_description/meshes/stl/Cover_Nose_Reals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 scale=0.001 0.001 0.001
- link rear_link: geometry collision box size=0.04 0.11 0.07; visual mesh filename=package://spotmicro_description/meshes/stl/B_cover.stl scale=0.001 0.001 0.001
Joints:
- added joint d435_color_joint: type fixed, parent d435_link, child d435_color_frame, origin xyz=0 0.015 0 rpy=0 0 0
- added joint d435_color_optical_joint: type fixed, parent d435_color_frame, child d435_color_optical_frame, origin xyz=0 0 0 rpy=-1.57079632679 0 -1.57079632679
- added joint d435_depth_joint: type fixed, parent d435_link, child d435_depth_frame, origin xyz=0 0 0 rpy=0 0 0
- added joint d435_depth_optical_joint: type fixed, parent d435_depth_frame, child d435_depth_optical_frame, origin xyz=0 0 0 rpy=-1.57079632679 0 -1.57079632679
- added joint d435_infra1_joint: type fixed, parent d435_link, child d435_infra1_frame, origin xyz=0 0.0 0 rpy=0 0 0
- added joint d435_infra1_optical_joint: type fixed, parent d435_infra1_frame, child d435_infra1_optical_frame, origin xyz=0 0 0 rpy=-1.57079632679 0 -1.57079632679
- added joint d435_infra2_joint: type fixed, parent d435_link, child d435_infra2_frame, origin xyz=0 -0.05 0 rpy=0 0 0
- added joint d435_infra2_optical_joint: type fixed, parent d435_infra2_frame, child d435_infra2_optical_frame, origin xyz=0 0 0 rpy=-1.57079632679 0 -1.57079632679
- added joint d435_joint: type fixed, parent base_link, child d435_bottom_screw_frame, origin xyz=0.14 0 -0.03
- added joint d435_link_joint: type fixed, parent d435_bottom_screw_frame, child d435_link, origin xyz=0.0106 0.0175 0.0125 rpy=0 0 0
- added joint imu_joint: type fixed, parent base_link, child imu_link, origin xyz=0.02 -0.04 0 rpy=1.57 0 0

File: urdf/spotmicroai.urdf.xacro (robot description, xacro)
@@ -262,4 +262,7 @@
       </inertial>
    </link>
+   <gazebo reference="base_inertia">
+      <material>Gazebo/FlatBlack</material>
+   </gazebo>
    <joint name="base_inertia_joint" type="fixed">
       <parent link="base_link" />
@@ -269,7 +272,14 @@
       <visual>
          <geometry>
-            <mesh filename="package://spotmicro_description/meshes/stl/backpart.stl" scale="0.001 0.001 0.001" />
-         </geometry>
-         <origin rpy="0 0 3.1416" xyz="0.042 0.055 -0.0195" />
+            <mesh filename="package://spotmicro_description/meshes/stl/Cover_Rear_Plain.stl" scale="0.001 0.001 0.001" />
+         </geometry>
+         <origin rpy="0 1.57 0" xyz="-0.115 0 -0.006" />
+         <material name="yellow" />
+      </visual>
+      <visual>
+         <geometry>
+            <mesh filename="package://spotmicro_description/meshes/stl/B_cover.stl" scale="0.001 0.001 0.001" />
+         </geometry>
+         <origin rpy="1.57 0 3.1416" xyz="0 0 -0.04" />
          <material name="yellow" />
       </visual>
@@ -295,7 +305,7 @@
       <visual>
          <geometry>
-            <mesh filename="package://spotmicro_description/meshes/stl/frontpart.stl" scale="0.001 0.001 0.001" />
-         </geometry>
-         <origin rpy="0 0 3.1416" xyz="0.042 0.055 -0.0205" />
+            <mesh filename="package://spotmicro_description/meshes/stl/Cover_Nose_Realsense.STL" scale="0.001 0.001 0.001" />
+         </geometry>
+         <origin rpy="3.1416 0 0" xyz="0.13 -0.001 -0.01" />
          <material name="yellow" />
       </visual>
@@ -323,3 +333,6 @@
    <xacro:gen_full_leg_joint pos="rear_left" shiftx="-${shiftx}" shifty="${shifty}" shift="${shift}" left="true" />
    <xacro:gen_full_leg_joint pos="rear_right" shiftx="-${shiftx}" shifty="-${shifty}" shift="-${shift}" left="false" />
+   <!-- Accessories -->
+   <xacro:include filename="$(find spotmicro_description)/urdf/accessories.urdf.xacro" />
+   <xacro:accessories base_name="base_link"/>
 </robot>
