Commit message: Improve stability of Gazebo simulation

File: urdf/accessories.urdf.xacro (robot description, xacro)
@@ -2,4 +2,16 @@
 <robot xmlns:xacro="http://ros.org/wiki/xacro">
   <xacro:macro name="accessories" params="base_name" >
+    <!-- Hokuyo UTM-30LX  -->
+    <xacro:include filename="$(find hector_sensors_description)/urdf/hokuyo_utm30lx.urdf.xacro" />
+    <xacro:hokuyo_utm30lx
+        name="hokuyo"
+        parent="${base_name}"
+        ros_topic="scan"
+        update_rate="30"
+        ray_count="1040"
+        min_angle="130"
+        max_angle="-130" >
+        <origin xyz="0 0 0.04"/>
+    </xacro:hokuyo_utm30lx>
     <!-- Intel Realsense D435 -->
     <xacro:property name="d435_link_name" value="d435"/>

File: urdf/spotmicroai.urdf (robot description, URDF)
Before this commit: robot SpotMicroAI, 35 links, 34 joints
Links:
- removed link front_left_leg_link_cover
- removed link front_right_leg_link_cover
- removed link rear_left_leg_link_cover
- removed link rear_right_leg_link_cover
- added link hokuyo_frame, mass 0.270; collision box size=0.058 0.058 0.087; visual mesh filename=package://hector_sensors_description/meshes/hokuyo_utm30lx/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
- link base_inertia: mass 2.80 -> 2.8
- link front_left_foot_link: geometry collision box size=0.026 0.02 0.08; visual mesh filename=package://spotmicro_description/meshes/stl/lfoot.stl scale=0.001 0.001 0.001
- link front_left_leg_link: mass 0.15 -> 0.1; geometry collision box size=0.028 0.036 0.109; visual mesh filename=package://spotmicro_description/meshes/stl/larm.stl scale=0.001 0.001 0.001
- link front_left_shoulder_link: mass 0.10 -> 0.15
- link front_left_toe_link: mass 0.05 -> 0.1
- link front_link: mass 0.20 -> 0.15
- link front_right_foot_link: geometry collision box size=0.026 0.02 0.08; visual mesh filename=package://spotmicro_description/meshes/stl/rfoot.stl scale=0.001 0.001 0.001
- link front_right_leg_link: mass 0.15 -> 0.1; geometry collision box size=0.028 0.036 0.109; visual mesh filename=package://spotmicro_description/meshes/stl/rarm.stl scale=0.001 0.001 0.001
- link front_right_shoulder_link: mass 0.10 -> 0.15
- link front_right_toe_link: mass 0.05 -> 0.1
- link rear_left_foot_link: geometry collision box size=0.026 0.02 0.08; visual mesh filename=package://spotmicro_description/meshes/stl/lfoot.stl scale=0.001 0.001 0.001
- link rear_left_leg_link: mass 0.15 -> 0.1; geometry collision box size=0.028 0.036 0.109; visual mesh filename=package://spotmicro_description/meshes/stl/larm.stl scale=0.001 0.001 0.001
- link rear_left_shoulder_link: mass 0.10 -> 0.15
- link rear_left_toe_link: mass 0.05 -> 0.1
- link rear_link: mass 0.20 -> 0.15
- link rear_right_foot_link: geometry collision box size=0.026 0.02 0.08; visual mesh filename=package://spotmicro_description/meshes/stl/rfoot.stl scale=0.001 0.001 0.001
- link rear_right_leg_link: mass 0.15 -> 0.1; geometry collision box size=0.028 0.036 0.109; visual mesh filename=package://spotmicro_description/meshes/stl/rarm.stl scale=0.001 0.001 0.001
- link rear_right_shoulder_link: mass 0.10 -> 0.15
- link rear_right_toe_link: mass 0.05 -> 0.1
Joints:
- removed joint base_inertia_joint
- removed joint front_left_leg_cover_joint
- removed joint front_right_leg_cover_joint
- removed joint rear_left_leg_cover_joint
- removed joint rear_right_leg_cover_joint
- added joint base_link_to_base_inertia: type fixed, parent base_link, child base_inertia
- added joint hokuyo_joint: type fixed, parent base_link, child hokuyo_frame, origin xyz=0 0 0.04
- joint front_left_foot: limit lower=-2.59 upper=0.1 effort=1000.0 velocity=0.5 -> lower=-2.59 upper=0.1 effort=25.0 velocity=1.5
- joint front_left_leg: limit lower=-2.666 upper=1.548 effort=1000.0 velocity=0.5 -> lower=-2.666 upper=1.548 effort=25.0 velocity=1.5; origin xyz=0 0.055 0 rpy=0 0 0 -> xyz=0 0.055 0
- joint front_left_shoulder: limit lower=-0.548 upper=0.548 effort=1000.0 velocity=0.7 -> lower=-0.548 upper=0.548 effort=25.0 velocity=1.5
- joint front_right_foot: limit lower=-2.59 upper=0.1 effort=1000.0 velocity=0.5 -> lower=-2.59 upper=0.1 effort=25.0 velocity=1.5
- joint front_right_leg: limit lower=-2.666 upper=1.548 effort=1000.0 velocity=0.5 -> lower=-2.666 upper=1.548 effort=25.0 velocity=1.5; origin xyz=0 -0.055 0 rpy=0 0 0 -> xyz=0 -0.055 0
- joint front_right_shoulder: limit lower=-0.548 upper=0.548 effort=1000.0 velocity=0.7 -> lower=-0.548 upper=0.548 effort=25.0 velocity=1.5
- joint rear_left_foot: limit lower=-2.59 upper=0.1 effort=1000.0 velocity=0.5 -> lower=-2.59 upper=0.1 effort=25.0 velocity=1.5
- joint rear_left_leg: limit lower=-2.666 upper=1.548 effort=1000.0 velocity=0.5 -> lower=-2.666 upper=1.548 effort=25.0 velocity=1.5; origin xyz=0 0.055 0 rpy=0 0 0 -> xyz=0 0.055 0
- joint rear_left_shoulder: limit lower=-0.548 upper=0.548 effort=1000.0 velocity=0.7 -> lower=-0.548 upper=0.548 effort=25.0 velocity=1.5
- joint rear_right_foot: limit lower=-2.59 upper=0.1 effort=1000.0 velocity=0.5 -> lower=-2.59 upper=0.1 effort=25.0 velocity=1.5
- joint rear_right_leg: limit lower=-2.666 upper=1.548 effort=1000.0 velocity=0.5 -> lower=-2.666 upper=1.548 effort=25.0 velocity=1.5; origin xyz=0 -0.055 0 rpy=0 0 0 -> xyz=0 -0.055 0
- joint rear_right_shoulder: limit lower=-0.548 upper=0.548 effort=1000.0 velocity=0.7 -> lower=-0.548 upper=0.548 effort=25.0 velocity=1.5

File: urdf/spotmicroai.urdf.xacro (robot description, xacro)
@@ -1,32 +1,6 @@
 <?xml version="1.0" encoding="UTF-8"?>
 <robot xmlns:xacro="http://www.ros.org/wiki/xacro" name="SpotMicroAI">
-   <material name="yellow">
-      <color rgba="0.92 0.83 0.0 1" />
-   </material>
-   <material name="black">
-      <color rgba="0.1 0.1 0.1 1" />
-   </material>
-   <material name="grey">
-      <color rgba="0.6 0.6 0.6 1" />
-   </material>
-   <!-- Params -->
-   <xacro:property name="body_length" value="0.140" />
-   <xacro:property name="body_width" value="0.110" />
-   <xacro:property name="body_height" value="0.070" />
-   <xacro:property name="lidar_length" value="0.0985" />
-   <xacro:property name="lidar_width" value="0.0577" />
-   <xacro:property name="lidar_height" value="0.070" />
-   <xacro:property name="front_length" value="0.058" />
-   <xacro:property name="rear_length" value="0.040" />
-   <xacro:property name="shoulder_length" value="0.044" />
-   <xacro:property name="shoulder_width" value="0.038" />
-   <xacro:property name="leg_length" value="0.109" />
-   <xacro:property name="foot_length" value="0.13" />
-   <xacro:property name="toe_radius" value="0.020" />
-   <!--  <xacro:property name="toe_radius" value="0.014" /> -->
-   <xacro:property name="toe_width" value="0.020" />
-   <xacro:property name="shift" value="0.055" />
-   <xacro:property name="shiftx" value="0.093" />
-   <xacro:property name="shifty" value="0.0395" />
+   <xacro:include filename="$(find spotmicro_description)/urdf/include/inertias.urdf.xacro"/>
+   <xacro:include filename="$(find spotmicro_description)/urdf/include/properties.urdf.xacro"/>
    <!-- Macros -->
    <xacro:macro name="gen_shoulder" params="name left">
@@ -51,10 +25,6 @@
                <box size="${shoulder_length} ${shoulder_width} ${body_height}" />
             </geometry>
-            <origin rpy="0 0 0" xyz="0 0 0" />
          </collision>
-         <inertial>
-            <mass value="0.10" />
-            <inertia ixx="100" ixy="0" ixz="0" iyy="100" iyz="0" izz="100" />
-         </inertial>
+         <xacro:inertial_cuboid mass="${shoulder_mass}" x_length="${shoulder_length}" y_length="${shoulder_width}" z_length="${body_height}"/>
       </link>
    </xacro:macro>
@@ -65,6 +35,5 @@
          <axis xyz="1 0 0" />
          <origin rpy="0 0 0" xyz="${shiftx} ${shifty} 0" />
-         <limit effort="1000.0" velocity="0.7" lower="-0.548" upper="0.548"/>
-         <dynamics damping="0.0" friction="0.5" />
+         <limit effort="25.0" velocity="1.5" lower="-0.548" upper="0.548"/>
       </joint>
       <transmission name="${pos}_shoulder_trans">
@@ -80,9 +49,9 @@
    </xacro:macro>
    <xacro:macro name="gen_leg" params="name left">
-      <link name="${name}_cover">
+      <link name="${name}">
          <visual>
             <xacro:if value="${left}">
                <geometry>
-                  <mesh filename="package://spotmicro_description/meshes/stl/larm_cover.stl" scale="0.001 0.001 0.001" />
+                  <mesh filename="package://spotmicro_description/meshes/stl/larm.stl" scale="0.001 0.001 0.001" />
                </geometry>
                <origin rpy="0 0 3.1416" xyz="0.134 -0.04 -0.0095" />
@@ -90,4 +59,20 @@
             <xacro:unless value="${left}">
                <geometry>
+                  <mesh filename="package://spotmicro_description/meshes/stl/rarm.stl" scale="0.001 0.001 0.001" />
+               </geometry>
+               <origin rpy="0 0 3.1416" xyz="0.134 0.149 -0.0095" />
+            </xacro:unless>
+            <material name="black" />
+         </visual>
+         <!-- Visual cover -->
+         <visual>
+            <xacro:if value="${left}">
+               <geometry>
+                  <mesh filename="package://spotmicro_description/meshes/stl/larm_cover.stl" scale="0.001 0.001 0.001" />
+               </geometry>
+               <origin rpy="0 0 3.1416" xyz="0.134 -0.04 -0.0095" />
+            </xacro:if>
+            <xacro:unless value="${left}">
+               <geometry>
                   <mesh filename="package://spotmicro_description/meshes/stl/rarm_cover.stl" scale="0.001 0.001 0.001" />
                </geometry>
@@ -96,34 +81,21 @@
             <material name="yellow" />
          </visual>
+         <collision>
+            <origin xyz="0 0 -0.050" />
+            <geometry>
+               <box size="${leg_width} ${leg_height} ${leg_length}" />
+            </geometry>
+         </collision>
+         <xacro:inertial_cuboid_with_pose mass="${leg_mass}" x_length="${leg_width}" y_length="${leg_height}" z_length="${leg_length}">
+            <origin xyz="0 0 -0.050" />
+         </xacro:inertial_cuboid_with_pose>
       </link>
-      <link name="${name}">
-         <visual>
-            <xacro:if value="${left}">
-               <geometry>
-                  <mesh filename="package://spotmicro_description/meshes/stl/larm.stl" scale="0.001 0.001 0.001" />
-               </geometry>
-               <origin rpy="0 0 3.1416" xyz="0.134 -0.04 -0.0095" />
-            </xacro:if>
-            <xacro:unless value="${left}">
-               <geometry>
-                  <mesh filename="package://spotmicro_description/meshes/stl/rarm.stl" scale="0.001 0.001 0.001" />
-               </geometry>
-               <origin rpy="0 0 3.1416" xyz="0.134 0.149 -0.0095" />
-            </xacro:unless>
-            <material name="black" />
-         </visual>
-         <collision>
-            <origin rpy="0.0 0.0 0.0" xyz="0.0 0.0 -0.050" />
-            <geometry>
-               <box size="0.028 0.036 ${leg_length}" />
-            </geometry>
-         </collision>
-         <inertial>
-            <mass value="0.15" />
-            <inertia ixx="1000" ixy="0" ixz="0" iyy="1000" iyz="0" izz="1000" />
-         </inertial>
-      </link>
-      <gazebo reference="${name}_cover">
-         <material>Gazebo/ZincYellow</material>
+      <gazebo reference="${name}">
+         <kp>1000000.0</kp>
+         <kd>1.0</kd>
+         <mu1>0.8</mu1>
+         <mu2>0.8</mu2>
+         <maxVel>0.0</maxVel>
+         <minDepth>0.001</minDepth>
       </gazebo>
    </xacro:macro>
@@ -133,7 +105,6 @@
          <child link="${pos}_leg_link" />
          <axis xyz="0 1 0" />
-         <origin rpy="0 0 0" xyz="0 ${shift} 0" />
-         <limit effort="1000.0" velocity="0.5" lower="-2.666" upper="1.548"/>
-         <dynamics damping="0.0" friction="0.0" />
+         <origin xyz="0 ${shift} 0" />
+         <limit effort="25.0" velocity="1.5" lower="-2.666" upper="1.548"/>
       </joint>
       <transmission name="${pos}_leg_trans">
@@ -147,9 +118,4 @@
          </actuator>
       </transmission>
-      <joint name="${pos}_leg_cover_joint" type="fixed">
-         <parent link="${pos}_leg_link" />
-         <child link="${pos}_leg_link_cover" />
-         <origin xyz="0 0 0" />
-      </joint>
    </xacro:macro>
    <xacro:macro name="gen_foot" params="name left">
@@ -172,12 +138,11 @@
          <collision>
             <geometry>
-               <box size="0.026 0.020 ${foot_length}" />
-            </geometry>
-            <origin rpy="0.0 0.0 0.0" xyz="0.0 0.0 -0.050" />
+               <box size="${foot_height} ${foot_width} ${foot_length}" />
+            </geometry>
+            <origin xyz="0 0 -0.050" />
          </collision>
-         <inertial>
-            <mass value="0.1" />
-            <inertia ixx="1000" ixy="0" ixz="0" iyy="1000" iyz="0" izz="1000" />
-         </inertial>
+         <xacro:inertial_cuboid_with_pose mass="${foot_mass}" x_length="${foot_height}" y_length="${foot_width}" z_length="${foot_length}">
+            <origin xyz="0 0 -0.050" />
+         </xacro:inertial_cuboid_with_pose>
       </link>
    </xacro:macro>
@@ -188,6 +153,5 @@
          <axis xyz="0 1 0" />
          <origin rpy="0 0 0" xyz="0.014 0 -${leg_length}" />
-         <limit effort="1000.0" velocity="0.5" lower="-2.59" upper="0.1"/>
-         <dynamics damping="0.0" friction="0.5" />
+         <limit effort="25.0" velocity="1.5" lower="-2.59" upper="0.1"/>
       </joint>
       <transmission name="${pos}_foot_trans">
@@ -215,12 +179,15 @@
                <sphere radius="${toe_radius}" />
             </geometry>
-            <origin rpy="0 0 0" xyz="0 0 0" />
-            <contact_coefficients mu="1.1" />
          </collision>
-         <inertial>
-            <mass value="0.05" />
-            <inertia ixx="1000" ixy="0" ixz="0" iyy="1000" iyz="0" izz="1000" />
-         </inertial>
+         <xacro:inertial_sphere mass="${toe_mass}" diameter="${2*toe_radius}"/>
       </link>
+      <gazebo reference="${name}">
+         <kp>1000000.0</kp>
+         <kd>1.0</kd>
+         <mu1>1.0</mu1>
+         <mu2>1.0</mu2>
+         <maxVel>0.0</maxVel>
+         <minDepth>0.001</minDepth>
+      </gazebo>
    </xacro:macro>
    <xacro:macro name="gen_toe_joint" params="pos">
@@ -228,5 +195,5 @@
          <parent link="${pos}_foot_link" />
          <child link="${pos}_toe_link" />
-         <origin xyz="0 0 -${foot_length}" />
+         <origin xyz="0 0 -0.13" />
       </joint>
    </xacro:macro>
@@ -255,15 +222,9 @@
             <box size="${body_length} ${body_width} ${body_height}" />
          </geometry>
-         <origin rpy="0 0 3.1416" xyz="0 0 0" />
+         <origin rpy="0 0 3.1416" />
       </collision>
-      <inertial>
-         <mass value="2.80" />
-         <inertia ixx="100" ixy="0" ixz="0" iyy="100" iyz="0" izz="100" />
-      </inertial>
+      <xacro:inertial_cuboid mass="${body_mass}" x_length="${body_length}" y_length="${body_width}" z_length="${body_height}"/>
    </link>
-   <gazebo reference="base_inertia">
-      <material>Gazebo/FlatBlack</material>
-   </gazebo>
-   <joint name="base_inertia_joint" type="fixed">
+   <joint name="base_link_to_base_inertia" type="fixed">
       <parent link="base_link" />
       <child link="base_inertia" />
@@ -288,10 +249,9 @@
             <box size="${rear_length} ${body_width} ${body_height}" />
          </geometry>
-         <origin rpy="0 0 0" xyz="-0.135 0 0" />
+         <origin xyz="-0.135 0 0" />
       </collision>
-      <inertial>
-         <mass value="0.20" />
-         <inertia ixx="100" ixy="0" ixz="0" iyy="100" iyz="0" izz="100" />
-      </inertial>
+      <xacro:inertial_cuboid_with_pose mass="${rear_mass}" x_length="${rear_length}" y_length="${body_width}" z_length="${body_height}">
+         <origin xyz="-0.135 0 0" />
+      </xacro:inertial_cuboid_with_pose>
    </link>
    <joint name="base_rear" type="fixed">
@@ -314,10 +274,9 @@
             <box size="${front_length} ${body_width} ${body_height}" />
          </geometry>
-         <origin rpy="0 0 0" xyz="0.135 0 0" />
+         <origin xyz="0.135 0 0" />
       </collision>
-      <inertial>
-         <mass value="0.20" />
-         <inertia ixx="100" ixy="0" ixz="0" iyy="100" iyz="0" izz="100" />
-      </inertial>
+      <xacro:inertial_cuboid_with_pose mass="${front_mass}" x_length="${front_length}" y_length="${body_width}" z_length="${body_height}">
+         <origin xyz="0.135 0 0" />
+      </xacro:inertial_cuboid_with_pose>
    </link>
    <gazebo reference="front_link">
@@ -336,3 +295,20 @@
    <xacro:include filename="$(find spotmicro_description)/urdf/accessories.urdf.xacro" />
    <xacro:accessories base_name="base_link"/>
+   <gazebo>
+      <plugin name="p3d_base_controller" filename="libgazebo_ros_p3d.so">
+            <alwaysOn>true</alwaysOn>
+            <updateRate>10.0</updateRate>
+            <bodyName>base_link</bodyName>
+            <topicName>odom/ground_truth</topicName>
+            <gaussianNoise>0.01</gaussianNoise>
+            <frameName>world</frameName>
+            <xyzOffsets>0 0 0</xyzOffsets>
+            <rpyOffsets>0 0 0</rpyOffsets>
+        </plugin>
+   </gazebo>
+   <gazebo>
+      <plugin name="gazebo_ros_control" filename="libgazebo_ros_control.so">
+         <legacyModeNS>true</legacyModeNS>
+      </plugin>
+   </gazebo>
 </robot>
