Commit message: Update URDF model

File: urdf/accessories.urdf.xacro (robot description, xacro)
@@ -57,4 +57,21 @@
     </gazebo>
     <!-- IMU MPU9250 -->
+    <link name="imu_link">
+      <xacro:dummy_inertia/>
+    </link>
+    <gazebo reference="imu_link">
+      <gravity>true</gravity>
+      <material>Gazebo/BlueGlow</material>
+    </gazebo>
+    <joint name="imu_joint" type="fixed">
+      <parent link="${base_name}" />
+      <child link="imu_link" />
+      <origin xyz="0.02 -0.04 0" rpy="1.57 0 0"/>
+    </joint>
+    <gazebo reference="imu_joint">
+      <provideFeedback>true</provideFeedback>
+      <disableFixedJointLumping>true</disableFixedJointLumping>
+      <preserveFixedJoint>true</preserveFixedJoint>
+    </gazebo>
     <gazebo>
       <plugin name="imu_controller" filename="libhector_gazebo_ros_imu.so">
@@ -70,10 +87,4 @@
       </plugin>
     </gazebo>
-    <link name="imu_link"/>
-    <joint name="imu_joint" type="fixed">
-      <parent link="${base_name}" />
-      <child link="imu_link" />
-      <origin xyz="0.02 -0.04 0" rpy="1.57 0 0"/>
-    </joint>
   </xacro:macro>
 </robot>

File: urdf/include/properties.urdf.xacro (robot description, xacro)
@@ -17,18 +17,18 @@
 <xacro:property name="body_mass"       value="2.800"/>
 <xacro:property name="front_length"    value="0.058" />
-<xacro:property name="front_mass"      value="0.150"/>
+<xacro:property name="front_mass"      value="0.30"/>
 <xacro:property name="rear_length"     value="0.040" />
-<xacro:property name="rear_mass"       value="0.150"/>
+<xacro:property name="rear_mass"       value="0.30"/>
 <xacro:property name="shoulder_length" value="0.044" />
 <xacro:property name="shoulder_width"  value="0.038" />
-<xacro:property name="shoulder_mass"   value="0.150"/>
+<xacro:property name="shoulder_mass"   value="0.30"/>
 <xacro:property name="leg_length"      value="0.109" />
 <xacro:property name="leg_width"       value="0.028"/>
 <xacro:property name="leg_height"      value="0.036"/>
-<xacro:property name="leg_mass"        value="0.100"/>
+<xacro:property name="leg_mass"        value="0.150"/>
 <xacro:property name="foot_length"     value="0.080" />
 <xacro:property name="foot_width"      value="0.020"/>
 <xacro:property name="foot_height"     value="0.026"/>
-<xacro:property name="foot_mass"       value="0.100"/>
+<xacro:property name="foot_mass"       value="0.150"/>
 <xacro:property name="toe_radius"      value="0.020" />
 <xacro:property name="toe_mass"        value="0.10" />
@@ -36,3 +36,6 @@
 <xacro:property name="shiftx"          value="0.093" />
 <xacro:property name="shifty"          value="0.0395" />
+<!-- Dynamics -->
+<xacro:property name="velocity"        value="1.5" />
+<xacro:property name="effort_limit"    value="5.0" />
 </robot>

File: urdf/spotmicroai.urdf (robot description, URDF)
Before this commit: robot SpotMicroAI, 32 links, 31 joints
Links:
- link front_left_foot_link: mass 0.1 -> 0.15
- link front_left_leg_link: mass 0.1 -> 0.15
- link front_left_shoulder_link: mass 0.15 -> 0.3
- link front_link: mass 0.15 -> 0.3
- link front_right_foot_link: mass 0.1 -> 0.15
- link front_right_leg_link: mass 0.1 -> 0.15
- link front_right_shoulder_link: mass 0.15 -> 0.3
- link imu_link: mass None -> 0.001
- link rear_left_foot_link: mass 0.1 -> 0.15
- link rear_left_leg_link: mass 0.1 -> 0.15
- link rear_left_shoulder_link: mass 0.15 -> 0.3
- link rear_link: mass 0.15 -> 0.3
- link rear_right_foot_link: mass 0.1 -> 0.15
- link rear_right_leg_link: mass 0.1 -> 0.15
- link rear_right_shoulder_link: mass 0.15 -> 0.3
Joints:
- joint front_left_foot: limit lower=-2.59 upper=0.1 effort=25.0 velocity=1.5 -> lower=-2.59 upper=0.1 effort=5.0 velocity=1.5
- joint front_left_leg: limit lower=-2.666 upper=1.548 effort=25.0 velocity=1.5 -> lower=-2.666 upper=1.548 effort=5.0 velocity=1.5
- joint front_left_shoulder: limit lower=-0.548 upper=0.548 effort=25.0 velocity=1.5 -> lower=-0.548 upper=0.548 effort=5.0 velocity=1.5
- joint front_right_foot: limit lower=-2.59 upper=0.1 effort=25.0 velocity=1.5 -> lower=-2.59 upper=0.1 effort=5.0 velocity=1.5
- joint front_right_leg: limit lower=-2.666 upper=1.548 effort=25.0 velocity=1.5 -> lower=-2.666 upper=1.548 effort=5.0 velocity=1.5
- joint front_right_shoulder: limit lower=-0.548 upper=0.548 effort=25.0 velocity=1.5 -> lower=-0.548 upper=0.548 effort=5.0 velocity=1.5
- joint rear_left_foot: limit lower=-2.59 upper=0.1 effort=25.0 velocity=1.5 -> lower=-2.59 upper=0.1 effort=5.0 velocity=1.5
- joint rear_left_leg: limit lower=-2.666 upper=1.548 effort=25.0 velocity=1.5 -> lower=-2.666 upper=1.548 effort=5.0 velocity=1.5
- joint rear_left_shoulder: limit lower=-0.548 upper=0.548 effort=25.0 velocity=1.5 -> lower=-0.548 upper=0.548 effort=5.0 velocity=1.5
- joint rear_right_foot: limit lower=-2.59 upper=0.1 effort=25.0 velocity=1.5 -> lower=-2.59 upper=0.1 effort=5.0 velocity=1.5
- joint rear_right_leg: limit lower=-2.666 upper=1.548 effort=25.0 velocity=1.5 -> lower=-2.666 upper=1.548 effort=5.0 velocity=1.5
- joint rear_right_shoulder: limit lower=-0.548 upper=0.548 effort=25.0 velocity=1.5 -> lower=-0.548 upper=0.548 effort=5.0 velocity=1.5

File: urdf/spotmicroai.urdf.xacro (robot description, xacro)
@@ -28,4 +28,8 @@
          <xacro:inertial_cuboid mass="${shoulder_mass}" x_length="${shoulder_length}" y_length="${shoulder_width}" z_length="${body_height}"/>
       </link>
+      <gazebo reference="${name}">
+         <mu1>100000.0</mu1>
+         <mu2>100000.0</mu2>
+      </gazebo>
    </xacro:macro>
    <xacro:macro name="gen_shoulder_joint" params="pos shiftx shifty">
@@ -35,5 +39,6 @@
          <axis xyz="1 0 0" />
          <origin rpy="0 0 0" xyz="${shiftx} ${shifty} 0" />
-         <limit effort="25.0" velocity="1.5" lower="-0.548" upper="0.548"/>
+         <limit effort="${effort_limit}" velocity="${velocity}" lower="-0.548" upper="0.548"/>
+         <dynamics friction="0.0" />
       </joint>
       <transmission name="${pos}_shoulder_trans">
@@ -92,10 +97,7 @@
       </link>
       <gazebo reference="${name}">
-         <kp>1000000.0</kp>
-         <kd>1.0</kd>
-         <mu1>0.8</mu1>
-         <mu2>0.8</mu2>
-         <maxVel>0.0</maxVel>
-         <minDepth>0.001</minDepth>
+         <mu1>100000.0</mu1>
+         <mu2>100000.0</mu2>
+         <material>Gazebo/Black</material>
       </gazebo>
    </xacro:macro>
@@ -106,5 +108,6 @@
          <axis xyz="0 1 0" />
          <origin xyz="0 ${shift} 0" />
-         <limit effort="25.0" velocity="1.5" lower="-2.666" upper="1.548"/>
+         <limit effort="${effort_limit}" velocity="${velocity}" lower="-2.666" upper="1.548"/>
+         <dynamics friction="0.0" />
       </joint>
       <transmission name="${pos}_leg_trans">
@@ -146,4 +149,8 @@
          </xacro:inertial_cuboid_with_pose>
       </link>
+      <gazebo reference="${name}">
+         <mu1>100000.0</mu1>
+         <mu2>100000.0</mu2>
+      </gazebo>
    </xacro:macro>
    <xacro:macro name="gen_foot_joint" params="pos">
@@ -153,5 +160,6 @@
          <axis xyz="0 1 0" />
          <origin rpy="0 0 0" xyz="0.014 0 -${leg_length}" />
-         <limit effort="25.0" velocity="1.5" lower="-2.59" upper="0.1"/>
+         <limit effort="${effort_limit}" velocity="${velocity}" lower="-2.59" upper="0.1"/>
+         <dynamics friction="0.0" />
       </joint>
       <transmission name="${pos}_foot_trans">
@@ -183,10 +191,26 @@
       </link>
       <gazebo reference="${name}">
-         <kp>1000000.0</kp>
-         <kd>1.0</kd>
-         <mu1>1.0</mu1>
-         <mu2>1.0</mu2>
-         <maxVel>0.0</maxVel>
-         <minDepth>0.001</minDepth>
+         <minDepth>0.0002</minDepth>
+         <collision name="${name}_collision_1">
+            <geometry>
+               <sphere>
+                  <radius>${toe_radius}</radius>
+               </sphere>
+            </geometry>
+            <surface>
+               <friction>
+                  <ode>
+                  <mu>100000.0</mu>
+                  <mu2>100000.0</mu2>
+                  </ode>
+                  <torsional>
+                  <coefficient>1000000</coefficient>
+                  <use_patch_radius>true</use_patch_radius>
+                  <surface_radius>${toe_radius}</surface_radius>
+                  <patch_radius>${toe_radius}</patch_radius>
+                  </torsional>
+               </friction>
+            </surface>
+         </collision>
       </gazebo>
    </xacro:macro>
@@ -197,4 +221,8 @@
          <origin xyz="0 0 -0.13" />
       </joint>
+      <gazebo reference="${pos}_toe">
+         <provideFeedback>true</provideFeedback>
+         <disableFixedJointLumping>true</disableFixedJointLumping>
+      </gazebo>
    </xacro:macro>
    <xacro:macro name="gen_full_leg_joint" params="pos shiftx shifty shift left">
@@ -226,8 +254,16 @@
       <xacro:inertial_cuboid mass="${body_mass}" x_length="${body_length}" y_length="${body_width}" z_length="${body_height}"/>
    </link>
+   <gazebo reference="base_inertia">
+      <mu1>100000.0</mu1>
+      <mu2>100000.0</mu2>
+   </gazebo>
    <joint name="base_link_to_base_inertia" type="fixed">
       <parent link="base_link" />
       <child link="base_inertia" />
    </joint>
+   <gazebo reference="base_link_to_base_inertia">
+      <provideFeedback>true</provideFeedback>
+      <disableFixedJointLumping>true</disableFixedJointLumping>
+  </gazebo>
    <link name="rear_link">
       <visual>
